Commit message: Add urdf and meshes

File: urdf/mini_bdx.urdf (robot description, URDF)
Before this commit: robot bdx-mini, 19 links, 18 joints
Links:
- link head_assembly: mass 0.500764 -> 0.561259; geometry collision mesh filename=package://mini_bdx_description/meshes/antenna.stl; collision mesh filename=package://mini_bdx_description/meshes/antenna.stl
- link knee_and_ankle_assembly: mass 0.113725 -> 0.118109; geometry collision mesh filename=package://mini_bdx_description/meshes/drive_palonier.stl; collision mesh filename=package://mini_bdx_description/meshes/left_knee_to_ankle_le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
- link knee_and_ankle_assembly_3: mass 0.113725 -> 0.118109; geometry collision mesh filename=package://mini_bdx_description/meshes/drive_palonier.stl; collision mesh filename=package://mini_bdx_description/meshes/left_knee_to_ankle_le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
- link trunk_assembly: mass 0.923001 -> 1.02895; geometry collision mesh filename=package://mini_bdx_description/meshes/back_panel.stl; collision mesh filename=package://mini_bdx_description/meshes/bno055.stl
Joints:
- joint head_pitch: limit lower=0 upper=1.5708 effort=10 velocity=10 -> lower=-0.785398 upper=0.785398 effort=10 velocity=10; origin xyz=-2.95597e-15 0.066 -6.93889e-18 rpy=-3.51457e-17 -1.44851e-16 -0.785398 -> xyz=5.20417e-18 0.066 -6.93889e-18 rpy=-1.19636e-16 3.97006e-18 -9.08773e-15
- joint head_roll: origin xyz=0.04095 6.11219e-18 -0.01915 rpy=-6.7987e-30 -1.5708 0 -> xyz=0.04095 3.39979e-16 -0.01915 rpy=1.17527e-16 -1.5708 0
- joint head_yaw: origin xyz=-1.38778e-17 0.057 0.01905 rpy=-1.5708 2.30638e-23 6.12323e-17 -> xyz=-1.6263e-17 0.057 0.01905 rpy=-1.5708 -2.83246e-15 -2.77679e-28
- joint imu_frame: origin xyz=-0.08711 1.249e-16 0.0422909 rpy=-5.43077e-16 1.41608e-16 -1.98935e-15 -> xyz=-0.08692 0.00079 0.0422909 rpy=1.26181e-15 -1.15513e-14 2.53967e-15
- joint left_ankle: limit lower=-0.785398 upper=2.35619 effort=10 velocity=10 -> lower=-1.5708 upper=1.5708 effort=10 velocity=10; origin xyz=-2.77556e-17 -0.07865 0.0001 rpy=6.89149e-27 9.32069e-29 -0.785398 -> xyz=0 -0.07865 0.0001 rpy=-2.69788e-17 -4.26045e-20 -5.55112e-17
- joint left_foot_frame: origin xyz=0.0005 -0.036225 0.01955 rpy=-1.5708 -1.45644e-30 0 -> xyz=0.0005 -0.036225 0.01955 rpy=-1.5708 -1.24631e-30 -1.77096e-25
- joint left_hip_pitch: limit lower=-0.436332 upper=1.309 effort=10 velocity=10 -> lower=-1.22173 upper=0.523599 effort=10 velocity=10; origin xyz=0.07415 1.45012e-17 0.03511 rpy=-1.5708 0.785398 1.5708 -> xyz=0.07415 3.81693e-16 0.03511 rpy=3.14159 1.5708 0
- joint left_hip_roll: origin xyz=0.01905 1.0339e-14 -0.046015 rpy=-1.5708 1.64593e-13 1.5708 -> xyz=0.01905 1.30035e-14 -0.046015 rpy=-1.5708 1.10442e-13 1.5708
- joint left_hip_yaw: origin xyz=-0.019 0.035 0.0459409 rpy=2.80971e-15 -2.15335e-14 1.96149e-13 -> xyz=-0.019 0.035 0.0457409 rpy=2.04385e-15 -1.12182e-14 9.65318e-16
- joint left_knee: limit lower=-3.14159 upper=2.22045e-16 effort=10 velocity=10 -> lower=-1.5708 upper=1.5708 effort=10 velocity=10; origin xyz=3.1225e-17 -0.07865 0.0001 rpy=-4.90788e-27 -2.64138e-16 1.5708 -> xyz=2.84495e-16 -0.07865 0.0001 rpy=-3.01789e-17 4.26046e-20 -1.98404e-12
- joint neck_pitch: limit lower=-1.13446 upper=0.349066 effort=10 velocity=10 -> lower=-0.349066 upper=1.13446 effort=10 velocity=10; origin xyz=0.001 0.01915 0.0900009 rpy=1.5708 -0.785398 8.65959e-17 -> xyz=0.001 0.01915 0.0900009 rpy=1.5708 -3.14089e-14 2.62734e-15
- joint right_ankle: limit lower=-0.785398 upper=2.35619 effort=10 velocity=10 -> lower=-1.5708 upper=1.5708 effort=10 velocity=10; origin xyz=-1.38778e-17 -0.07865 0.0001 rpy=-1.69496e-15 5.11604e-16 -0.785398 -> xyz=-8.32667e-17 -0.07865 0.0001 rpy=1.88569e-26 -1.01508e-25 2.06793e-26
- joint right_foot_frame: origin xyz=0.0005 -0.036225 0.01955 rpy=-1.5708 2.77556e-17 -5.55112e-17 -> xyz=0.0005 -0.036225 0.01955 rpy=-1.5708 9.68789e-29 0
- joint right_hip_pitch: limit lower=-1.309 upper=0.436332 effort=10 velocity=10 -> lower=-0.523599 upper=1.22173 effort=10 velocity=10; origin xyz=-0.07415 -1.99764e-17 0.03511 rpy=1.5708 0.785398 1.5708 -> xyz=-0.07415 1.76562e-16 0.03511 rpy=-1.40962e-15 1.5708 0
- joint right_hip_roll: origin xyz=0.01905 5.77038e-14 -0.046015 rpy=-1.5708 4.8633e-13 1.5708 -> xyz=0.01905 5.9841e-14 -0.046015 rpy=-1.5708 -1.07345e-13 1.5708
- joint right_hip_yaw: origin xyz=-0.019 -0.035 0.0459409 rpy=-2.95717e-16 -2.22045e-14 -7.55636e-15 -> xyz=-0.019 -0.035 0.0457409 rpy=2.06672e-15 -1.15513e-14 1.93627e-13
- joint right_knee: limit lower=-3.14159 upper=6.51035e-13 effort=10 velocity=10 -> lower=-1.5708 upper=1.5708 effort=10 velocity=10; origin xyz=-6.93889e-18 0.07865 0.037 rpy=-3.14159 -3.99728e-16 -1.5708 -> xyz=-4.16334e-17 0.07865 0.037 rpy=-3.14159 -2.18222e-26 3.06314e-17

Commit message: Rename package

File: urdf/mini_bdx.urdf (robot description, URDF)
Before this commit: robot bdx-mini, 19 links, 18 joints
Links:
- link foot_assembly: geometry collision mesh filename=package://open_duck_mini_description/meshes/foot_bottom_pla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; collision mesh filename=package://open_duck_mini_description/meshes/foot_bottom_tpu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
- link foot_assembly_2: geometry collision mesh filename=package://open_duck_mini_description/meshes/foot_bottom_pla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; collision mesh filename=package://open_duck_mini_description/meshes/foot_bottom_tpu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
- link head_assembly: geometry collision mesh filename=package://open_duck_mini_description/meshes/antenna.stl; collision mesh filename=package://open_duck_mini_description/meshes/antenna.stl
- link head_pitch_to_yaw: geometry collision mesh filename=package://open_duck_mini_description/meshes/head_pitch_to_y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; visual mesh filename=package://open_duck_mini_description/meshes/head_pitch_to_y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
- link hip_roll_assembly: geometry collision mesh filename=package://open_duck_mini_description/meshes/drive_palonier.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; collision mesh filename=package://open_duck_mini_description/meshes/passive_palonie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
- link hip_roll_assembly_2: geometry collision mesh filename=package://open_duck_mini_description/meshes/drive_palonier.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; collision mesh filename=package://open_duck_mini_description/meshes/passive_palonie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
- link knee_and_ankle_assembly: geometry collision mesh filename=package://open_duck_mini_description/meshes/drive_palonier.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; collision mesh filename=package://open_duck_mini_description/meshes/left_knee_to_an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
- link knee_and_ankle_assembly_2: geometry collision mesh filename=package://open_duck_mini_description/meshes/drive_palonier.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; collision mesh filename=package://open_duck_mini_description/meshes/left_knee_to_an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
- link knee_and_ankle_assembly_3: geometry collision mesh filename=package://open_duck_mini_description/meshes/drive_palonier.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; collision mesh filename=package://open_duck_mini_description/meshes/left_knee_to_an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
- link knee_and_ankle_assembly_4: geometry collision mesh filename=package://open_duck_mini_description/meshes/drive_palonier.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; collision mesh filename=package://open_duck_mini_description/meshes/left_knee_to_an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
- link left_roll_to_pitch_assembly: geometry collision mesh filename=package://open_duck_mini_description/meshes/drive_palonier.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; collision mesh filename=package://open_duck_mini_description/meshes/left_roll_to_pi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
- link neck_pitch_assembly: geometry collision mesh filename=package://open_duck_mini_description/meshes/drive_palonier.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; collision mesh filename=package://open_duck_mini_description/meshes/neck_left_sheet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
- link neck_yaw_assembly: geometry collision mesh filename=package://open_duck_mini_description/meshes/drive_palonier.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; collision mesh filename=package://open_duck_mini_description/meshes/head_yaw_to_rol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
- link right_roll_to_pitch_assembly: geometry collision mesh filename=package://open_duck_mini_description/meshes/drive_palonier.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; collision mesh filename=package://open_duck_mini_description/meshes/passive_palonie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
- link trunk_assembly: geometry collision mesh filename=package://open_duck_mini_description/meshes/back_panel.stl; collision mesh filename=package://open_duck_mini_description/meshes/bno055.stl
